File: Delay/SingleDelay.kicad_sch (KiCad schematic)
At the start: 54 parts, among them J201 AudioJack2_SwitchT, J202 AudioJack2_SwitchT, J203 AudioJack2_SwitchT, Q201 2N3904, U101 TL072, U102 TL072, U103 TL072, U104 TL072, U105 TL072, U106 TL072, U201 PT2399

Commit message: Add delay daisy chaining switches and readme
Parts:
- removed J202, J203: AudioJack2_SwitchT, symbol Connector:AudioJack2_SwitchT
Connections:
- net In: now reaches R207.1
- net Out: now reaches R223.1
- no-connect marks 4 -> 2

Commit message: Finish delay PCB
Parts:
- added C417, C418, C419, C420, C421, C422: 0.1u, Capacitor_THT:C_Disc_D5.0mm_W2.5mm_P5.00mm, symbol Device:C
- added U401, U402, U403: TL072, Package_DIP:DIP-8_W7.62mm_Socket, symbol Amplifier_Operational:TL072
- C401: renamed from C201; footprint (none) -> Capacitor_THT:C_Disc_D5.0mm_W2.5mm_P5.00mm
- C402: renamed from C202; footprint (none) -> Capacitor_THT:CP_Radial_D5.0mm_P2.00mm
- C403: renamed from C203; footprint (none) -> Capacitor_THT:C_Disc_D5.0mm_W2.5mm_P5.00mm
- C404: renamed from C204; footprint (none) -> Capacitor_THT:C_Disc_D5.0mm_W2.5mm_P5.00mm
- C405: renamed from C205; footprint (none) -> Capacitor_THT:CP_Radial_D5.0mm_P2.00mm
- C406: renamed from C206; footprint (none) -> Capacitor_THT:C_Disc_D5.0mm_W2.5mm_P5.00mm
- C407: renamed from C207; footprint (none) -> Capacitor_THT:C_Disc_D5.0mm_W2.5mm_P5.00mm
- C408: renamed from C208; footprint (none) -> Capacitor_THT:C_Disc_D5.0mm_W2.5mm_P5.00mm
- C409: renamed from C209; footprint (none) -> Capacitor_THT:C_Disc_D5.0mm_W2.5mm_P5.00mm
- C410: renamed from C210; footprint (none) -> Capacitor_THT:C_Disc_D5.0mm_W2.5mm_P5.00mm
- C411: renamed from C211; footprint (none) -> Capacitor_THT:C_Disc_D5.0mm_W2.5mm_P5.00mm
- C412: renamed from C212; footprint (none) -> Capacitor_THT:C_Disc_D5.0mm_W2.5mm_P5.00mm
- C413: renamed from C213; footprint (none) -> Capacitor_THT:C_Disc_D5.0mm_W2.5mm_P5.00mm
- C414: renamed from C214; footprint (none) -> Capacitor_THT:C_Disc_D5.0mm_W2.5mm_P5.00mm
- C415: renamed from C215; footprint (none) -> Capacitor_THT:C_Disc_D5.0mm_W2.5mm_P5.00mm; symbol Device:C_Polarized -> Device:C
- C416: renamed from C216; footprint (none) -> Capacitor_THT:C_Disc_D5.0mm_W2.5mm_P5.00mm; symbol Device:C_Polarized -> Device:C
- J401: renamed from J201; footprint (none) -> Connector_Audio:Jack_3.5mm_QingPu_WQP-PJ398SM_Vertical_CircularHoles
- Q401: renamed from Q201; footprint Package_TO_SOT_THT:TO-92_Inline -> Package_TO_SOT_THT:TO-92_HandSolder
- RV401: renamed from RV201; footprint (none) -> Potentiometer_THT:Potentiometer_Alpha_RD901F-40-00D_Single_Vertical_CircularHoles
- RV402: renamed from RV202; footprint (none) -> Potentiometer_THT:Potentiometer_Alpha_RD901F-40-00D_Single_Vertical_CircularHoles
- RV403: renamed from RV203; footprint (none) -> Potentiometer_THT:Potentiometer_Alpha_RD901F-40-00D_Single_Vertical_CircularHoles
- U401: renamed from U101; footprint (none) -> Package_DIP:DIP-8_W7.62mm_Socket
- U401: renamed from U102; footprint (none) -> Package_DIP:DIP-8_W7.62mm_Socket
- U402: renamed from U103; footprint (none) -> Package_DIP:DIP-8_W7.62mm_Socket
- U402: renamed from U104; footprint (none) -> Package_DIP:DIP-8_W7.62mm_Socket
- U403: renamed from U105; footprint (none) -> Package_DIP:DIP-8_W7.62mm_Socket
- U403: renamed from U106; footprint (none) -> Package_DIP:DIP-8_W7.62mm_Socket
- U404: renamed from U201; footprint (none) -> Package_DIP:DIP-16_W7.62mm_Socket
- renumbered D201 to D401, R201 to R401, R202 to R402, R203 to R403, R204 to R404, R205 to R405, R206 to R406, R207 to R407, R208 to R408, R209 to R409, R210 to R410, R211 to R411, R212 to R412, R213 to R413, R214 to R414, R215 to R415, R216 to R416, R217 to R417, R218 to R418, R219 to R419, R220 to R420, R221 to R421, R222 to R422, R223 to R423
Connections:
- net +12V: now also C417.1, C419.1, C421.1
- net GND: now also C417.2, C418.1, C419.2, C420.1, C421.2, C422.1
- new net -12V: C418.2, C420.2, C422.2
