File: Power Supply/Panel/Panel.kicad_pcb (KiCad board)
At the start: 2 copper layers, 40.3 x 128.5 mm, 0 parts

Commit message: Add SKVCF
Changed lines of the file:
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@@
     (effects (font (size 1 1) (thickness 0.15)) (justify mirror))
   )
-  (gr_text "On" (at 144.35 138.7) (layer "F.Mask")
+  (gr_text "On" (at 144.35 138.7) (layer "F.SilkS")
     (effects (font (size 2.5 2.5) (thickness 0.25)))
   )
-  (gr_text "+12V" (at 151.35 70.2) (layer "F.Mask")
+  (gr_text "+12V" (at 151.35 70.2) (layer "F.SilkS")
     (effects (font (size 2.5 2.5) (thickness 0.25)))
   )
-  (gr_text "Off" (at 158.35 138.7) (layer "F.Mask")
+  (gr_text "Off" (at 158.35 138.7) (layer "F.SilkS")
     (effects (font (size 2.5 2.5) (thickness 0.25)))
   )
-  (gr_text "-12V" (at 151.35 93.033333) (layer "F.Mask")
+  (gr_text "-12V" (at 151.35 93.033333) (layer "F.SilkS")
     (effects (font (size 2.5 2.5) (thickness 0.25)))
   )
-  (gr_text "Power" (at 151.35 45.2) (layer "F.Mask")
+  (gr_text "Power" (at 151.35 45.2) (layer "F.SilkS")
     (effects (font (size 8 8) (thickness 1.2)))
   )
-  (gr_text "+5V" (at 151.35 115.866667) (layer "F.Mask")
+  (gr_text "+5V" (at 151.35 115.866667) (layer "F.SilkS")
     (effects (font (size 2.5 2.5) (thickness 0.25)))
   )
