File: Simplified Controller/Out.kicad_sch (KiCad schematic)
At the start: 44 parts

Commit message: Finish simplified controller
Parts:
- gave numbers to parts that had none: 44

Commit message: Add SKVCF
Connections:
- net +5V: no longer U201.8 (VREFIN)
- new net +5VA: U201.8 (VREFIN)
Changed lines of the file:
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@@
   (junction (at 212.09 72.39) (diameter 0) (color 0 0 0 0)
   )
+  (junction (at 36.83 72.39) (diameter 0) (color 0 0 0 0)
+  )
   (junction (at 212.09 46.99) (diameter 0) (color 0 0 0 0)
   )
   (junction (at 36.83 105.41) (diameter 0) (color 0 0 0 0)
-  )
-  (junction (at 36.83 72.39) (diameter 0) (color 0 0 0 0)
   )
   (no_connect (at 214.63 82.55))
@@
     (stroke (width 0) (type default) (color 0 0 0 0))
   )
+  (wire (pts (xy 36.83 72.39) (xy 38.1 72.39))
+    (stroke (width 0) (type default) (color 0 0 0 0))
+  )
   (wire (pts (xy 46.99 100.33) (xy 49.53 100.33))
     (stroke (width 0) (type default) (color 0 0 0 0))
@@
   )
   (wire (pts (xy 57.15 39.37) (xy 99.06 39.37))
-    (stroke (width 0) (type default) (color 0 0 0 0))
-  )
-  (wire (pts (xy 36.83 72.39) (xy 38.1 72.39))
     (stroke (width 0) (type default) (color 0 0 0 0))
   )
@@
     (pin "1")
   )
+  (symbol (lib_id "power:+5VA") (at 26.67 90.17 90) (unit 1)
+    (in_bom yes) (on_board yes) (fields_autoplaced)
+    (property "Reference" "#PWR0204" (id 0) (at 30.48 90.17 0)
+      (effects (font (size 1.27 1.27)) hide)
+    )
+    (property "Value" "+5VA" (id 1) (at 22.86 90.1699 90)
+      (effects (font (size 1.27 1.27)) (justify left))
+    )
+    (property "Footprint" "" (id 2) (at 26.67 90.17 0)
+      (effects (font (size 1.27 1.27)) hide)
+    )
+    (property "Datasheet" "" (id 3) (at 26.67 90.17 0)
+      (effects (font (size 1.27 1.27)) hide)
+    )
+    (pin "1")
+  )
   (symbol (lib_id "Connector:AudioJack2_SwitchT") (at 172.72 46.99 180) (unit 1)
     (in_bom yes) (on_board yes)
@@
     (pin "1")
   )
+  (symbol (lib_id "power:+5V") (at 36.83 72.39 0) (unit 1)
+    (in_bom yes) (on_board yes) (fields_autoplaced)
+    (property "Reference" "#PWR0205" (id 0) (at 36.83 76.2 0)
+      (effects (font (size 1.27 1.27)) hide)
+    )
+    (property "Value" "+5V" (id 1) (at 36.83 67.31 0))
+    (property "Footprint" "" (id 2) (at 36.83 72.39 0)
+      (effects (font (size 1.27 1.27)) hide)
+    )
+    (property "Datasheet" "" (id 3) (at 36.83 72.39 0)
+      (effects (font (size 1.27 1.27)) hide)
+    )
+    (pin "1")
+  )
   (symbol (lib_id "Device:R") (at 266.7 59.69 270) (unit 1)
     (in_bom yes) (on_board yes)
@@
     (pin "1")
   )
-  (symbol (lib_id "power:+5V") (at 36.83 72.39 0) (unit 1)
-    (in_bom yes) (on_board yes)
-    (property "Reference" "#PWR0205" (id 0) (at 36.83 76.2 0)
-      (effects (font (size 1.27 1.27)) hide)
-    )
-    (property "Value" "+5V" (id 1) (at 37.211 67.9958 0))
-    (property "Footprint" "" (id 2) (at 36.83 72.39 0)
-      (effects (font (size 1.27 1.27)) hide)
-    )
-    (property "Datasheet" "" (id 3) (at 36.83 72.39 0)
-      (effects (font (size 1.27 1.27)) hide)
-    )
-    (pin "1")
-  )
   (symbol (lib_id "Connector:AudioJack2_SwitchT") (at 219.71 135.89 180) (unit 1)
     (in_bom yes) (on_board yes)
@@
       (effects (font (size 1.27 1.27)) hide)
     )
-    (pin "1")
-  )
-  (symbol (lib_id "power:+5V") (at 26.67 90.17 90) (unit 1)
-    (in_bom yes) (on_board yes)
-    (property "Reference" "#PWR0204" (id 0) (at 30.48 90.17 0)
-      (effects (font (size 1.27 1.27)) hide)
-    )
-    (property "Value" "+5V" (id 1) (at 22.2758 89.789 0))
-    (property "Footprint" "" (id 2) (at 26.67 90.17 0)
-      (effects (font (size 1.27 1.27)) hide)
-    )
-    (property "Datasheet" "" (id 3) (at 26.67 90.17 0)
-      (effects (font (size 1.27 1.27)) hide)
-    )
