File: Simplified Controller/Panel/Panel.kicad_pcb (KiCad board)
At the start: 2 copper layers, 182.5 x 128.5 mm, 0 parts

Commit message: Add SKVCF
Changed lines of the file:
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@@
       (layerselection 0x00010fc_ffffffff)
       (disableapertmacros false)
-      (usegerberextensions false)
-      (usegerberattributes true)
-      (usegerberadvancedattributes true)
-      (creategerberjobfile true)
+      (usegerberextensions true)
+      (usegerberattributes false)
+      (usegerberadvancedattributes false)
+      (creategerberjobfile false)
       (svguseinch false)
       (svgprecision 6)
@@
       (psa4output false)
       (plotreference true)
-      (plotvalue true)
+      (plotvalue false)
       (plotinvisibletext false)
       (sketchpadsonfab false)
-      (subtractmaskfromsilk false)
+      (subtractmaskfromsilk true)
       (outputformat 1)
       (mirror false)
-      (drillshape 1)
+      (drillshape 0)
       (scaleselection 1)
-      (outputdirectory "")
+      (outputdirectory "gerbers/")
     )
   )
@@
     (effects (font (size 1 1) (thickness 0.15)) (justify mirror))
   )
-  (gr_text "Trigger" (at 222.7 138.885714) (layer "F.Mask")
+  (gr_text "Trigger" (at 222.7 138.885714) (layer "F.SilkS")
     (effects (font (size 2.5 2.5) (thickness 0.25)))
   )
-  (gr_text "Output" (at 192.7 84.135715) (layer "F.Mask")
+  (gr_text "Output" (at 192.7 84.135715) (layer "F.SilkS")
     (effects (font (size 2.5 2.5) (thickness 0.25)))
   )
-  (gr_text "1V/Oct" (at 222.7 113.6) (layer "F.Mask")
+  (gr_text "1V/Oct" (at 222.7 113.6) (layer "F.SilkS")
     (effects (font (size 2.5 2.5) (thickness 0.25)))
   )
-  (gr_text "Channel" (at 208.7 84.135715) (layer "F.Mask")
+  (gr_text "Channel" (at 208.7 84.135715) (layer "F.SilkS")
     (effects (font (size 2.5 2.5) (thickness 0.25)))
   )
-  (gr_text "MIDI Interface" (at 148.3 45.385715) (layer "F.Mask")
+  (gr_text "MIDI Interface" (at 148.3 45.385715) (layer "F.SilkS")
     (effects (font (size 10 10) (thickness 1.2)))
   )
-  (gr_text "Gate" (at 222.7 126.242857) (layer "F.Mask")
+  (gr_text "Gate" (at 222.7 126.242857) (layer "F.SilkS")
     (effects (font (size 2.5 2.5) (thickness 0.25)))
   )
-  (gr_text "MIDI In" (at 73.925 119.135715) (layer "F.Mask")
+  (gr_text "MIDI In" (at 73.925 119.135715) (layer "F.SilkS")
     (effects (font (size 2.5 2.5) (thickness 0.25)))
   )
