File: VCA/Panel/Panel.kicad_pcb (KiCad board)
At the start: 2 copper layers, 91.3 x 128.5 mm, 0 parts

Commit message: Add SKVCF
Changed lines of the file:
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@@
   )
   (net 0 "")
+  (gr_line (start 151.5 107.2) (end 168.9 107.2) (layer "F.SilkS") (width 0.5))
+  (gr_line (start 151.5 58.8) (end 168.9 58.8) (layer "F.SilkS") (width 0.5))
   (gr_circle (center 123.95 58.7) (end 127.55 58.7) (layer "B.Mask") (width 5) (fill none))
   (gr_circle (center 109.8 31.7) (end 111.4 31.7) (layer "B.Mask") (width 2) (fill none))
@@
   (gr_circle (center 186 31.7) (end 187.6 31.7) (layer "B.Mask") (width 2) (fill none))
   (gr_circle (center 123.95 127.2) (end 127.55 127.2) (layer "B.Mask") (width 5) (fill none))
-  (gr_line (start 151.5 107.2) (end 168.9 107.2) (layer "F.Mask") (width 0.5))
   (gr_circle (center 147.95 58.7) (end 151.55 58.7) (layer "F.Mask") (width 5) (fill none))
   (gr_circle (center 123.95 107.2) (end 127.55 107.2) (layer "F.Mask") (width 5) (fill none))
@@
   (gr_circle (center 123.95 78.7) (end 127.55 78.7) (layer "F.Mask") (width 5) (fill none))
   (gr_circle (center 109.8 154.2) (end 111.4 154.2) (layer "F.Mask") (width 2) (fill none))
-  (gr_line (start 151.5 58.8) (end 168.9 58.8) (layer "F.Mask") (width 0.5))
   (gr_circle (center 147.95 107.2) (end 151.55 107.2) (layer "F.Mask") (width 5) (fill none))
   (gr_circle (center 186 154.2) (end 187.6 154.2) (layer "F.Mask") (width 2) (fill none))
@@
     (effects (font (size 1 1) (thickness 0.15)) (justify mirror))
   )
-  (gr_text "Line Out" (at 171.95 137.2) (layer "F.Mask")
+  (gr_text "Line Out" (at 171.95 137.2) (layer "F.SilkS")
     (effects (font (size 2.5 2.5) (thickness 0.3)))
   )
-  (gr_text "Line Out" (at 171.95 88.7) (layer "F.Mask")
+  (gr_text "Line Out" (at 171.95 88.7) (layer "F.SilkS")
     (effects (font (size 2.5 2.5) (thickness 0.3)))
   )
-  (gr_text "In" (at 123.95 88.7) (layer "F.Mask")
+  (gr_text "In" (at 123.95 88.7) (layer "F.SilkS")
     (effects (font (size 2.5 2.5) (thickness 0.3)))
   )
-  (gr_text "Out" (at 147.95 88.7) (layer "F.Mask")
+  (gr_text "Out" (at 147.95 88.7) (layer "F.SilkS")
     (effects (font (size 2.5 2.5) (thickness 0.3)))
   )
-  (gr_text "Level" (at 147.95 117.2) (layer "F.Mask")
+  (gr_text "Level" (at 147.95 117.2) (layer "F.SilkS")
     (effects (font (size 2.5 2.5) (thickness 0.3)))
   )
-  (gr_text "In" (at 123.95 137.2) (layer "F.Mask")
+  (gr_text "In" (at 123.95 137.2) (layer "F.SilkS")
     (effects (font (size 2.5 2.5) (thickness 0.3)))
   )
-  (gr_text "Out" (at 147.95 137.2) (layer "F.Mask")
+  (gr_text "Out" (at 147.95 137.2) (layer "F.SilkS")
     (effects (font (size 2.5 2.5) (thickness 0.3)))
   )
-  (gr_text "VCA" (at 147.95 43.7) (layer "F.Mask")
+  (gr_text "VCA" (at 147.95 43.7) (layer "F.SilkS")
     (effects (font (size 10 10) (thickness 1.2)))
   )
-  (gr_text "Level" (at 147.95 68.7) (layer "F.Mask")
+  (gr_text "Level" (at 147.95 68.7) (layer "F.SilkS")
     (effects (font (size 2.5 2.5) (thickness 0.3)))
   )
