File: VCF/Panel/Panel.kicad_pcb (KiCad board)
At the start: 2 copper layers, 111.4 x 128.5 mm, 0 parts

Commit message: Add SKVCF
Changed lines of the file:
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@@
   )
   (net 0 "")
+  (gr_line (start 146 112.3) (end 146 132.7) (layer "F.SilkS") (width 0.5))
+  (gr_line (start 146 63.8) (end 146 84.2) (layer "F.SilkS") (width 0.5))
+  (gr_line (start 170 63.8) (end 170 84.2) (layer "F.SilkS") (width 0.5))
   (gr_circle (center 170 112.3) (end 173.6 112.3) (layer "B.Mask") (width 5) (fill none))
   (gr_circle (center 146 132.3) (end 149.6 132.3) (layer "B.Mask") (width 5) (fill none))
@@
   (gr_circle (center 146 112.3) (end 149.6 112.3) (layer "B.Mask") (width 5) (fill none))
   (gr_circle (center 170 132.3) (end 173.6 132.3) (layer "B.Mask") (width 5) (fill none))
-  (gr_line (start 146 112.3) (end 146 132.7) (layer "F.Mask") (width 0.5))
   (gr_circle (center 170 83.8) (end 173.6 83.8) (layer "F.Mask") (width 5) (fill none))
   (gr_circle (center 170 112.3) (end 173.6 112.3) (layer "F.Mask") (width 5) (fill none))
   (gr_circle (center 146 63.8) (end 149.6 63.8) (layer "F.Mask") (width 5) (fill none))
   (gr_circle (center 170 63.8) (end 173.6 63.8) (layer "F.Mask") (width 5) (fill none))
-  (gr_line (start 146 63.8) (end 146 84.2) (layer "F.Mask") (width 0.5))
   (gr_circle (center 194.32 36.8) (end 195.92 36.8) (layer "F.Mask") (width 2) (fill none))
   (gr_circle (center 122 122.3) (end 125.6 122.3) (layer "F.Mask") (width 5) (fill none))
   (gr_circle (center 170 132.3) (end 173.6 132.3) (layer "F.Mask") (width 5) (fill none))
-  (gr_line (start 170 63.8) (end 170 84.2) (layer "F.Mask") (width 0.5))
   (gr_circle (center 122 73.8) (end 125.6 73.8) (layer "F.Mask") (width 5) (fill none))
   (gr_circle (center 97.8 159.3) (end 99.4 159.3) (layer "F.Mask") (width 2) (fill none))
@@
     (effects (font (size 1 1) (thickness 0.15)) (justify mirror))
   )
-  (gr_text "Resonance" (at 134 142.3) (layer "F.Mask")
+  (gr_text "Resonance" (at 134 142.3) (layer "F.SilkS")
     (effects (font (size 2.5 2.5) (thickness 0.25)))
   )
-  (gr_text "Out" (at 170 142.3) (layer "F.Mask")
+  (gr_text "Out" (at 170 142.3) (layer "F.SilkS")
     (effects (font (size 2.5 2.5) (thickness 0.25)))
   )
-  (gr_text "VCLPF" (at 146 48.8) (layer "F.Mask")
+  (gr_text "VCLPF" (at 146 48.8) (layer "F.SilkS")
     (effects (font (size 10 10) (thickness 1.2)))
   )
-  (gr_text "Transistor\nLadder" (at 184.133333 48.8) (layer "F.Mask")
+  (gr_text "Transistor\nLadder" (at 184.133333 48.8) (layer "F.SilkS")
     (effects (font (size 2.5 2.5) (thickness 0.25)))
   )
-  (gr_text "Cutoff" (at 146 93.8) (layer "F.Mask")
+  (gr_text "Cutoff" (at 146 93.8) (layer "F.SilkS")
     (effects (font (size 2.5 2.5) (thickness 0.25)))
   )
-  (gr_text "In" (at 170 122.3) (layer "F.Mask")
+  (gr_text "In" (at 170 122.3) (layer "F.SilkS")
     (effects (font (size 2.5 2.5) (thickness 0.25)))
   )
