File: VCO/Panel/Panel.kicad_pcb (KiCad board)
At the start: 2 copper layers, 162.2 x 128.5 mm, 1 part

Commit message: Add SKVCF
Other:
- board text added: "VCO2"
- board text removed: "VCO"
Changed lines of the file:
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@@
         (xy -2.004338 -2.126664)
         (xy -1.956136 -2.124537)
-      ) (layer "F.Mask") (width 0.01) (fill solid))
+      ) (layer "F.SilkS") (width 0.01) (fill solid))
   )
+  (gr_line (start 187.3 57) (end 205.5 57) (layer "F.SilkS") (width 0.5))
+  (gr_line (start 187.3 77) (end 205.5 77) (layer "F.SilkS") (width 0.5))
+  (gr_line (start 103.1 105.5) (end 118.1 125.5) (layer "F.SilkS") (width 0.5))
+  (gr_line (start 208.1 105.5) (end 208.1 125.5) (layer "F.SilkS") (width 0.5))
+  (gr_line (start 204.1 133.5) (end 212.1 137.5) (layer "F.SilkS") (width 0.25))
+  (gr_line (start 204.1 133.5) (end 204.1 137.5) (layer "F.SilkS") (width 0.25))
+  (gr_line (start 148.1 105.5) (end 148.1 125.5) (layer "F.SilkS") (width 0.5))
+  (gr_line (start 152.1 137.5) (end 152.1 135.5) (layer "F.SilkS") (width 0.25))
+  (gr_line (start 115.2 77) (end 133.4 77) (layer "F.SilkS") (width 0.5))
+  (gr_line (start 148.1 133.5) (end 148.1 137.5) (layer "F.SilkS") (width 0.25))
+  (gr_line (start 90.1 137.5) (end 92.1 135.5) (layer "F.SilkS") (width 0.25))
+  (gr_line (start 84.1 135.5) (end 86.1 133.5) (layer "F.SilkS") (width 0.25))
+  (gr_line (start 103.1 105.5) (end 88.1 125.5) (layer "F.SilkS") (width 0.5))
+  (gr_line (start 182.1 133.5) (end 182.1 137.5) (layer "F.SilkS") (width 0.25))
+  (gr_line (start 144.1 135.5) (end 144.1 133.5) (layer "F.SilkS") (width 0.25))
+  (gr_line (start 86.1 133.5) (end 90.1 137.5) (layer "F.SilkS") (width 0.25))
+  (gr_line (start 144.1 133.5) (end 148.1 133.5) (layer "F.SilkS") (width 0.25))
+  (gr_line (start 174.1 137.5) (end 182.1 133.5) (layer "F.SilkS") (width 0.25))
+  (gr_line (start 178.1 105.5) (end 178.1 125.5) (layer "F.SilkS") (width 0.5))
+  (gr_line (start 148.1 137.5) (end 152.1 137.5) (layer "F.SilkS") (width 0.25))
   (gr_circle (center 88.1 57) (end 91.7 57) (layer "B.Mask") (width 5) (fill none))
   (gr_circle (center 148.1 125.5) (end 151.7 125.5) (layer "B.Mask") (width 5) (fill none))
@@
   (gr_circle (center 112.1 57) (end 115.7 57) (layer "B.Mask") (width 5) (fill none))
   (gr_circle (center 118.1 125.5) (end 121.7 125.5) (layer "B.Mask") (width 5) (fill none))
-  (gr_line (start 187.3 57) (end 205.5 57) (layer "F.Mask") (width 0.5))
-  (gr_line (start 187.3 77) (end 205.5 77) (layer "F.Mask") (width 0.5))
-  (gr_line (start 103.1 105.5) (end 118.1 125.5) (layer "F.Mask") (width 0.5))
-  (gr_line (start 208.1 105.5) (end 208.1 125.5) (layer "F.Mask") (width 0.5))
-  (gr_line (start 204.1 133.5) (end 212.1 137.5) (layer "F.Mask") (width 0.25))
-  (gr_line (start 204.1 133.5) (end 204.1 137.5) (layer "F.Mask") (width 0.25))
-  (gr_line (start 148.1 105.5) (end 148.1 125.5) (layer "F.Mask") (width 0.5))
   (gr_circle (center 208.1 125.5) (end 211.7 125.5) (layer "F.Mask") (width 5) (fill none))
-  (gr_line (start 152.1 137.5) (end 152.1 135.5) (layer "F.Mask") (width 0.25))
   (gr_circle (center 148.1 125.5) (end 151.7 125.5) (layer "F.Mask") (width 5) (fill none))
-  (gr_line (start 115.2 77) (end 133.4 77) (layer "F.Mask") (width 0.5))
   (gr_circle (center 160.1 67) (end 163.7 67) (layer "F.Mask") (width 5) (fill none))
   (gr_circle (center 208.1 57) (end 211.7 57) (layer "F.Mask") (width 5) (fill none))
   (gr_circle (center 178.1 125.5) (end 181.7 125.5) (layer "F.Mask") (width 5) (fill none))
-  (gr_line (start 148.1 133.5) (end 148.1 137.5) (layer "F.Mask") (width 0.25))
   (gr_circle (center 118.1 125.5) (end 121.7 125.5) (layer "F.Mask") (width 5) (fill none))
   (gr_circle (center 184.1 57) (end 187.7 57) (layer "F.Mask") (width 5) (fill none))
-  (gr_line (start 90.1 137.5) (end 92.1 135.5) (layer "F.Mask") (width 0.25))
   (gr_circle (center 136.1 57) (end 139.7 57) (layer "F.Mask") (width 5) (fill none))
   (gr_circle (center 88.1 77) (end 91.7 77) (layer "F.Mask") (width 5) (fill none))
   (gr_circle (center 208.1 77) (end 211.7 77) (layer "F.Mask") (width 5) (fill none))
-  (gr_line (start 84.1 135.5) (end 86.1 133.5) (layer "F.Mask") (width 0.25))
-  (gr_line (start 103.1 105.5) (end 88.1 125.5) (layer "F.Mask") (width 0.5))
-  (gr_line (start 182.1 133.5) (end 182.1 137.5) (layer "F.Mask") (width 0.25))
   (gr_circle (center 88.1 57) (end 91.7 57) (layer "F.Mask") (width 5) (fill none))
   (gr_circle (center 221.82 152.5) (end 223.42 152.5) (layer "F.Mask") (width 2) (fill none))
   (gr_circle (center 88.1 125.5) (end 91.7 125.5) (layer "F.Mask") (width 5) (fill none))
   (gr_circle (center 184.1 77) (end 187.7 77) (layer "F.Mask") (width 5) (fill none))
-  (gr_line (start 144.1 135.5) (end 144.1 133.5) (layer "F.Mask") (width 0.25))
   (gr_circle (center 74.5 152.5) (end 76.1 152.5) (layer "F.Mask") (width 2) (fill none))
-  (gr_line (start 86.1 133.5) (end 90.1 137.5) (layer "F.Mask") (width 0.25))
-  (gr_line (start 144.1 133.5) (end 148.1 133.5) (layer "F.Mask") (width 0.25))
-  (gr_line (start 174.1 137.5) (end 182.1 133.5) (layer "F.Mask") (width 0.25))
   (gr_circle (center 74.5 30) (end 76.1 30) (layer "F.Mask") (width 2) (fill none))
-  (gr_line (start 178.1 105.5) (end 178.1 125.5) (layer "F.Mask") (width 0.5))
   (gr_circle (center 112.1 57) (end 115.7 57) (layer "F.Mask") (width 5) (fill none))
   (gr_circle (center 221.82 30) (end 223.42 30) (layer "F.Mask") (width 2) (fill none))
-  (gr_line (start 148.1 137.5) (end 152.1 137.5) (layer "F.Mask") (width 0.25))
   (gr_circle (center 112.1 77) (end 115.7 77) (layer "F.Mask") (width 5) (fill none))
   (gr_circle (center 136.1 77) (end 139.7 77) (layer "F.Mask") (width 5) (fill none))
@@
     (effects (font (size 1 1) (thickness 0.15)) (justify mirror))
   )
-  (gr_text "Linear FM" (at 196.1 87) (layer "F.Mask")
+  (gr_text "Linear FM" (at 196.1 87) (layer "F.SilkS")
     (effects (font (size 2.5 2.5) (thickness 0.25)))
   )
-  (gr_text "Fast" (at 160.1 57) (layer "F.Mask")
+  (gr_text "Fast" (at 160.1 57) (layer "F.SilkS")
     (effects (font (size 2.5 2.5) (thickness 0.25)))
   )
-  (gr_text "Slow" (at 160.1 77) (layer "F.Mask")
+  (gr_text "Slow" (at 160.1 77) (layer "F.SilkS")
     (effects (font (size 2.5 2.5) (thickness 0.25)))
   )
-  (gr_text "Fine" (at 112.1 67) (layer "F.Mask")
+  (gr_text "Fine" (at 112.1 67) (layer "F.SilkS")
     (effects (font (size 2.5 2.5) (thickness 0.25)))
   )
-  (gr_text "1V/Octave" (at 136.1 67) (layer "F.Mask")
+  (gr_text "1V/Octave" (at 136.1 67) (layer "F.SilkS")
     (effects (font (size 2.5 2.5) (thickness 0.25)))
   )
-  (gr_text "PWM" (at 112.1 87) (layer "F.Mask")
+  (gr_text "PWM" (at 112.1 87) (layer "F.SilkS")
     (effects (font (size 2.5 2.5) (thickness 0.25)))
   )
-  (gr_text "Exponential FM" (at 196.1 67) (layer "F.Mask")
+  (gr_text "Exponential FM" (at 196.1 67) (layer "F.SilkS")
     (effects (font (size 2.5 2.5) (thickness 0.25)))
   )
-  (gr_text "Coarse" (at 88.1 67) (layer "F.Mask")
+  (gr_text "Coarse" (at 88.1 67) (layer "F.SilkS")
     (effects (font (size 2.5 2.5) (thickness 0.25)))
   )
-  (gr_text "VCO" (at 148.1 42) (layer "F.Mask")
+  (gr_text "VCO2" (at 148.1 42) (layer "F.SilkS")
     (effects (font (size 10 10) (thickness 1.2)))
   )
