File: Envelope Generator/Out.kicad_sch (KiCad schematic)
At the start: 27 parts, among them J301 AudioJack2_SwitchT, J302 AudioJack2_SwitchT, J303 AudioJack2_SwitchT, J304 AudioJack2_SwitchT, U102 TL072, U103 TL072, U104 TL072

Commit message: New modules, small updates
Connections:
- net GND: now also U102.5 (+); no longer U102.3 (+)
- net at R301.2, RV302.1, RV302.2: now also U102.6 (-); no longer U102.2 (-)
- net at R303.1, R304.2, R305.2: now also U102.7; no longer U102.1
- net at R302.2, R303.2: now also U103.5 (+); no longer U103.3 (+)
- net at R307.1, R309.2, R310.2: now also U103.7, U104.5 (+); no longer U103.1, U104.3 (+)
- net at R306.1, R307.2: now also U103.6 (-); no longer U103.2 (-)
- new net: R313.2, U104.6 (-), U104.7
