File: Decay/Decay.kicad_sch (KiCad schematic)
At the start: 24 parts

Commit message: Update decay caps, fix ERC issues
Parts:
- C3, C5: renamed from C?; value 0.1u -> 10u
- C4, C6: renamed from C?; value 10n -> 0.1u
- gave numbers to parts that had none: 18
Connections:
- net Chasis is gone; now on net Chassis: J3.5 (Pin_5), J3.6 (Pin_6)
