File: Out/Line.kicad_sch (KiCad schematic)
At the start: 29 parts

Commit message: Fix out module ERC issues
Parts:
- C201, C202: renamed from C?; value 10n -> 0.1u
- gave numbers to parts that had none: 24

Commit message: Place PSU components on PCB
Parts:
- C201, C202, C203, C204, C205, C206, C207, C208: footprint (none) -> 0_Capacitor_THT:C_Disc_D5.5mm_W2.5mm_P2.50mm
- C209, C210, C211, C212: footprint (none) -> 0_Capacitor_THT:C_Disc_D5.5mm_W4.0mm_P2.50mm
- RV202: symbol Custom:R_Potentiometer_Dual_MountingPin -> 0_Device:R_Potentiometer_Dual_MountingPin
- U201: symbol Custom:NJM2068D -> 0_Amplifier_Operational:NJM2068D
Changed lines of the file:
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@@
     (effects (font (size 1.27 1.27)) (justify right))
   )
-  (symbol (lib_id "Custom:R_Potentiometer_Dual_MountingPin") (at 128.27 86.36 270) (mirror x) (unit 1)
+  (symbol (lib_id "0_Device:R_Potentiometer_Dual_MountingPin") (at 128.27 86.36 270) (mirror x) (unit 1)
     (in_bom yes) (on_board yes)
     (property "Reference" "RV202" (id 0) (at 120.65 80.0131 90))
@@
     (pin "6")
   )
-  (symbol (lib_id "Custom:Chassis") (at 198.12 74.93 0) (unit 1)
+  (symbol (lib_id "0_power:Chassis") (at 198.12 74.93 0) (unit 1)
     (in_bom no) (on_board no)
     (property "Reference" "#U0202" (id 0) (at 198.12 80.01 0)
@@
       (effects (font (size 1.27 1.27)) (justify left))
     )
-    (property "Footprint" "" (id 2) (at 171.45 53.6448 0)
+    (property "Footprint" "0_Capacitor_THT:C_Disc_D5.5mm_W2.5mm_P2.50mm" (id 2) (at 171.45 53.6448 0)
       (effects (font (size 1.27 1.27)) hide)
     )
@@
       (effects (font (size 1.27 1.27)) (justify left))
     )
-    (property "Footprint" "" (id 2) (at 162.2552 102.87 0)
+    (property "Footprint" "0_Capacitor_THT:C_Disc_D5.5mm_W2.5mm_P2.50mm" (id 2) (at 162.2552 102.87 0)
       (effects (font (size 1.27 1.27)) hide)
     )
@@
     (pin "1")
   )
-  (symbol (lib_name "NJM2068D_1") (lib_id "Custom:NJM2068D") (at 91.44 96.52 0) (unit 2)
+  (symbol (lib_id "0_Amplifier_Operational:NJM2068D") (at 91.44 96.52 0) (unit 2)
     (in_bom yes) (on_board yes) (fields_autoplaced)
     (property "Reference" "U201" (id 0) (at 91.44 87.7402 0))
@@
     (property "Reference" "C212" (id 0) (at 186.69 122.4112 90))
     (property "Value" "100u" (id 1) (at 186.69 124.9481 90))
-    (property "Footprint" "" (id 2) (at 190.5 127.3048 0)
+    (property "Footprint" "0_Capacitor_THT:C_Disc_D5.5mm_W4.0mm_P2.50mm" (id 2) (at 190.5 127.3048 0)
       (effects (font (size 1.27 1.27)) hide)
     )
@@
       (effects (font (size 1.27 1.27)) (justify right))
     )
-    (property "Footprint" "" (id 2) (at 89.2048 125.73 0)
+    (property "Footprint" "0_Capacitor_THT:C_Disc_D5.5mm_W2.5mm_P2.50mm" (id 2) (at 89.2048 125.73 0)
       (effects (font (size 1.27 1.27)) hide)
     )
@@
     (pin "2")
   )
-  (symbol (lib_name "NJM2068D_2") (lib_id "Custom:NJM2068D") (at 91.44 76.2 0) (unit 1)
+  (symbol (lib_id "0_Amplifier_Operational:NJM2068D") (at 91.44 76.2 0) (unit 1)
     (in_bom yes) (on_board yes) (fields_autoplaced)
     (property "Reference" "U201" (id 0) (at 91.44 67.4202 0))
@@
       (effects (font (size 1.27 1.27)) (justify left))
     )
-    (property "Footprint" "" (id 2) (at 162.2552 138.43 0)
+    (property "Footprint" "0_Capacitor_THT:C_Disc_D5.5mm_W2.5mm_P2.50mm" (id 2) (at 162.2552 138.43 0)
       (effects (font (size 1.27 1.27)) hide)
     )
@@
       (effects (font (size 1.27 1.27)) (justify right))
     )
-    (property "Footprint" "" (id 2) (at 89.2048 118.11 0)
+    (property "Footprint" "0_Capacitor_THT:C_Disc_D5.5mm_W2.5mm_P2.50mm" (id 2) (at 89.2048 118.11 0)
       (effects (font (size 1.27 1.27)) hide)
     )
@@
     (pin "1")
   )
-  (symbol (lib_id "Custom:Chassis") (at 198.12 130.81 0) (unit 1)
+  (symbol (lib_id "0_power:Chassis") (at 198.12 130.81 0) (unit 1)
     (in_bom no) (on_board no)
     (property "Reference" "#U0203" (id 0) (at 198.12 135.89 0)
@@
     (property "Reference" "C209" (id 0) (at 186.69 56.3712 90))
     (property "Value" "100u" (id 1) (at 186.69 58.9081 90))
-    (property "Footprint" "" (id 2) (at 190.5 61.2648 0)
+    (property "Footprint" "0_Capacitor_THT:C_Disc_D5.5mm_W4.0mm_P2.50mm" (id 2) (at 190.5 61.2648 0)
       (effects (font (size 1.27 1.27)) hide)
     )
@@
     (pin "2")
   )
-  (symbol (lib_id "Custom:NJM2068D") (at 96.52 125.73 0) (unit 3)
+  (symbol (lib_id "0_Amplifier_Operational:NJM2068D") (at 96.52 125.73 0) (unit 3)
     (in_bom yes) (on_board yes) (fields_autoplaced)
     (property "Reference" "U201" (id 0) (at 94.615 124.8953 0)
@@
     (property "Reference" "C211" (id 0) (at 186.69 112.2512 90))
     (property "Value" "100u" (id 1) (at 186.69 114.7881 90))
-    (property "Footprint" "" (id 2) (at 190.5 117.1448 0)
+    (property "Footprint" "0_Capacitor_THT:C_Disc_D5.5mm_W4.0mm_P2.50mm" (id 2) (at 190.5 117.1448 0)
       (effects (font (size 1.27 1.27)) hide)
     )
@@
     (pin "1")
   )
-  (symbol (lib_id "Custom:Chassis") (at 120.65 107.95 0) (unit 1)
+  (symbol (lib_id "0_power:Chassis") (at 120.65 107.95 0) (unit 1)
     (in_bom no) (on_board no)
     (property "Reference" "#U0201" (id 0) (at 120.65 113.03 0)
@@
       (effects (font (size 1.27 1.27)) (justify left))
     )
-    (property "Footprint" "" (id 2) (at 171.45 109.5248 0)
+    (property "Footprint" "0_Capacitor_THT:C_Disc_D5.5mm_W2.5mm_P2.50mm" (id 2) (at 171.45 109.5248 0)
       (effects (font (size 1.27 1.27)) hide)
     )
@@
       (effects (font (size 1.27 1.27)) (justify left))
     )
-    (property "Footprint" "" (id 2) (at 162.2552 46.99 0)
+    (property "Footprint" "0_Capacitor_THT:C_Disc_D5.5mm_W2.5mm_P2.50mm" (id 2) (at 162.2552 46.99 0)
       (effects (font (size 1.27 1.27)) hide)
     )
@@
     (property "Reference" "C210" (id 0) (at 186.69 66.5312 90))
     (property "Value" "100u" (id 1) (at 186.69 69.0681 90))
-    (property "Footprint" "" (id 2) (at 190.5 71.4248 0)
+    (property "Footprint" "0_Capacitor_THT:C_Disc_D5.5mm_W4.0mm_P2.50mm" (id 2) (at 190.5 71.4248 0)
       (effects (font (size 1.27 1.27)) hide)
     )
@@
       (effects (font (size 1.27 1.27)) (justify left))
     )
-    (property "Footprint" "" (id 2) (at 162.2552 82.55 0)
-      (effects (font (size 1.27 1.27)) hide)
-    )
+    (property "Footprint" "0_Capacitor_THT:C_Disc_D5.5mm_W2.5mm_P2.50mm" (id 2) (at 162.2552 82.55 0)
+      (effects (font (size 1.27 1.27)) hide)
+    )
