File: 13700 VCA/13700 VCA.kicad_pcb (KiCad board)
At the start: 2 copper layers, 81 parts, among them J101 Conn_02x05_Odd_Even, J102 AudioJack2_SwitchT, J103 AudioJack2_SwitchT, J104 AudioJack2_SwitchT, J105 AudioJack2_SwitchT, J106 AudioJack2_SwitchT, J107 AudioJack2_SwitchT, J108 AudioJack2_SwitchT, J201 AudioJack2_SwitchT, J202 AudioJack2_SwitchT, Q101 2N3906, Q102 2N3906, U101 LM13700, U102 TL072, U103 TL072, U201 TL072

Commit message: Create VCA front end project
Parts:
- Q101, Q102: footprint Package_TO_SOT_THT:TO-92_HandSolder -> Package_TO_SOT_THT:TO-92_Inline

Commit message: Finish VCA PCB
Parts:
- removed J102, J103, J104, J105, J106, J107, J108, J201, J202: AudioJack2_SwitchT, Connector_Audio:Jack_3.5mm_QingPu_WQP-PJ398SM_Vertical_CircularHoles
- removed R101, R102, R116, R117, R201: 47k, Resistor_THT:R_Axial_DIN0207_L6.3mm_D2.5mm_P7.62mm_Horizontal
- removed R103, R118: 15k, Resistor_THT:R_Axial_DIN0207_L6.3mm_D2.5mm_P7.62mm_Horizontal
- removed R105, R108, R120, R123: 100k, Resistor_THT:R_Axial_DIN0207_L6.3mm_D2.5mm_P7.62mm_Horizontal
- removed R202: 56k, Resistor_THT:R_Axial_DIN0207_L6.3mm_D2.5mm_P7.62mm_Horizontal
- removed RV101, RV102, RV104, RV105, RV201, RV202, RV203, RV204: 10k, 0_Potentiometer_THT:Potentiometer_Alpha_RD901F-40-00D_Single_Vertical_MP
- added H1: MNT_STANDOFF, 0_MountingHole:MountingHole_Pitch7.5mm_Drill3.4mm, F.Cu at (104.2, 129.9)
- added H2: MNT_STANDOFF, 0_MountingHole:MountingHole_Pitch7.5mm_Drill3.4mm, F.Cu at (143.2, 129.9)
- added J2: Conn_01x19, Connector_PinHeader_2.54mm:PinHeader_1x19_P2.54mm_Vertical, F.Cu at (123.7, 44.7)
- C101, C102, C103, C104, C105, C106, C107, C108, C109, C110, C111, C112, C201, C202, C203, C204, D101, D102, D103, D104, J101, R104, R106, R107, R109, R110, R111, R112, R113, R114, R115, R119, R121, R122, R124, R125, R126, R127, R128, R129, R130, R203, R204, R205, RV103, RV106, U101, U102, U103, U201: moved to B.Cu
- Q101, Q102: footprint Package_TO_SOT_THT:TO-92_Inline -> Package_TO_SOT_THT:TO-92_HandSolder; moved to B.Cu
- moved C202 116.7 mm to (86.8, 49.1), turned to -90 degrees
- moved C108 114.2 mm to (99.0, 68.8)
- moved D103 110.5 mm to (92.8, 75.0), turned to -90 degrees
- moved R204 109.5 mm to (86.5, 38.4), turned to -90 degrees
- moved R203 107.7 mm to (96.9, 37.5), turned to 180 degrees
- moved C201 105.4 mm to (92.5, 40.8), turned to 180 degrees
- moved C204 103.0 mm to (95.1, 54.9), turned to 180 degrees
- moved Q102 100.3 mm to (115.0, 82.8), turned to -90 degrees
- moved C103 96.3 mm to (95.8, 77.5), turned to -90 degrees
- moved C203 94.4 mm to (100.8, 44.0), turned to -90 degrees
- moved R205 92.7 mm to (97.7, 58.0), turned to 180 degrees
- moved R106 90.8 mm to (109.1, 50.0), turned to 180 degrees
- moved U201 90.7 mm to (90.0, 44.0), turned to -90 degrees
- moved C110 86.8 mm to (119.5, 121.4)
- moved U102 85.0 mm to (99.0, 80.0)
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Connections:
- net /Stereo Controls/CV_COMMON renamed /CV_COMMON
- net /Stereo Controls/CV_COMMON_OFFSET renamed /CV_COMMON_OFFSET
- net Net-(D103-K) renamed /CV_1
- net Net-(D104-K) renamed /CV_2
- net Net-(J105-PadT) renamed /OUT_1
- net Net-(J108-PadT) renamed /OUT_2
- net Net-(U101A--) renamed /IN_1
- net Net-(U101C--) renamed /IN_2
- net Net-(U201A--) renamed /PAN_CV
- J101 pad 2: +12V -> GND
- J101 pad 3: GND -> Chassis
- J101 pad 5: Chassis -> -12V
- J101 pad 6: Chassis -> +12V
- J101 pad 8: GND -> Chassis
- J101 pad 9: -12V -> GND
Routing:
- net +12V: track 0.00 -> 200.3 mm, vias 0 -> 5
- net -12V: track 0.00 -> 154.3 mm, vias 0 -> 7
- net /CV_1: track 0.00 -> 74.3 mm
- net /OUT_2: track 0.00 -> 55.6 mm
- net /OUT_1: track 0.00 -> 52.2 mm
- net /PAN_CV: track 0.00 -> 50.9 mm
- net /CV_2: track 0.00 -> 44.9 mm
- net /Stereo Controls/PAN_1: track 0.00 -> 31.5 mm
- net Net-(U103A--): track 0.00 -> 31.5 mm
- net Net-(U103B--): track 0.00 -> 28.8 mm
- net /IN_1: track 0.00 -> 24.2 mm
- net /Stereo Controls/PAN_2: track 0.00 -> 22.1 mm
- net /IN_2: track 0.00 -> 20.6 mm
- net Chassis: track 0.00 -> 19.4 mm
- net Net-(U201B--): track 0.00 -> 18.4 mm
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- added copper zone on B.Cu, net GND
Other:
- board outline added: 80.9 x 104.5 mm

Commit message: Add VCA and VCO front panels
Other:
- board text added: "JLCJLCJLCJLC"
- board text added: "VCA V1 Matthew Taylor Based on electricdruid.net LM13700 VCA"
Changed lines of the file:
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@@
 	)
 	(setup
+		(stackup
+			(layer "F.SilkS"
+				(type "Top Silk Screen")
+			)
+			(layer "F.Paste"
+				(type "Top Solder Paste")
+			)
+			(layer "F.Mask"
+				(type "Top Solder Mask")
+				(thickness 0.01)
+			)
+			(layer "F.Cu"
+				(type "copper")
+				(thickness 0.035)
+			)
+			(layer "dielectric 1"
+				(type "core")
+				(thickness 1.51)
+				(material "FR4")
+				(epsilon_r 4.5)
+				(loss_tangent 0.02)
+			)
+			(layer "B.Cu"
+				(type "copper")
+				(thickness 0.035)
+			)
+			(layer "B.Mask"
+				(type "Bottom Solder Mask")
+				(thickness 0.01)
+			)
+			(layer "B.Paste"
+				(type "Bottom Solder Paste")
+			)
+			(layer "B.SilkS"
+				(type "Bottom Silk Screen")
+			)
+			(copper_finish "None")
+			(dielectric_constraints no)
+		)
 		(pad_to_mask_clearance 0)
 		(allow_soldermask_bridges_in_footprints no)
@@
 		(tags "Resistor Axial_DIN0207 series Axial Horizontal pin pitch 7.62mm 0.25W = 1/4W length 6.3mm diameter 2.5mm")
 		(property "Reference" "R128"
-			(at 3.81119 0.01 270)
+			(at 3.81119 0.01 -90)
 			(layer "B.SilkS")
 			(effects
@@
 		)
 		(property "Value" "1k"
-			(at 3.81 -2.37 270)
+			(at 3.81 -2.37 -90)
 			(layer "B.Fab")
 			(effects
@@
 		)
 		(fp_text user "${REFERENCE}"
-			(at 3.81 0 270)
+			(at 3.81 0 -90)
 			(layer "B.Fab")
 			(effects
@@
 		(tags "to-92 sc-43 sc-43a sot54 PA33 transistor")
 		(property "Reference" "Q101"
-			(at 1.27 4 360)
+			(at 1.27 4 0)
 			(layer "B.SilkS")
 			(effects
@@
 		)
 		(property "Value" "2N3906"
-			(at 1.27 -2.79 360)
+			(at 1.27 -2.79 0)
 			(layer "B.Fab")
 			(effects
@@
 		)
 		(fp_text user "${REFERENCE}"
-			(at 1.27 0 360)
+			(at 1.27 0 0)
 			(layer "B.Fab")
 			(effects
@@
 		(layer "Edge.Cuts")
 	)
+	(gr_text "VCA V1\nMatthew Taylor\nBased on electricdruid.net LM13700 VCA"
+		(at 163 139 0)
+		(layer "B.SilkS")
+		(effects
+			(font
+				(size 1 1)
+				(thickness 0.15)
+			)
+			(justify left bottom mirror)
+		)
+	)
+	(gr_text "JLCJLCJLCJLC"
+		(at 151.5 137.75 0)
+		(layer "F.SilkS")
+		(effects
+			(font
+				(size 1 1)
+				(thickness 0.15)
+			)
+			(justify left bottom)
+		)
+	)
 	(segment

Commit message: Begin revised delay
Parts:
- added R4: 47k, Resistor_THT:R_Axial_DIN0207_L6.3mm_D2.5mm_P7.62mm_Horizontal, F.Cu at (171.9, 111.5)
- added R5: 47k, Resistor_THT:R_Axial_DIN0207_L6.3mm_D2.5mm_P7.62mm_Horizontal, F.Cu at (171.9, 115.5)
- J101: value Conn_02x05_Odd_Even -> Conn_02x05_Top_Bottom
Connections:
- net /Stereo Controls/PAN_1 renamed Net-(C201-Pad2)
- net /Stereo Controls/PAN_2 renamed Net-(C204-Pad2)
- RV103 pad 1: /IN_1 -> Net-(U101A--)
- RV106 pad 1: /IN_2 -> Net-(U101C--)
- U101 pad 13: /IN_1 -> Net-(U101A--)
- U101 pad 4: /IN_2 -> Net-(U101C--)

Commit message: PCB fixes and cleanup
Parts:
- R4, R5: moved to B.Cu
- moved R4 68.7 mm to (103.5, 104.7)
- moved R5 30.3 mm to (143.2, 105.8), turned to 180 degrees
Routing:
- net /IN_2: track 20.6 -> 30.7 mm, vias 0 -> 2
- net Net-(U101A--): track 0.00 -> 9.14 mm
- net Net-(U101C--): track 0.00 -> 8.77 mm
- net /IN_1: track 24.2 -> 32.3 mm, vias 0 -> 2
- net /OUT_1: track 52.2 -> 52.6 mm, vias 0 -> 2
