File: 13700 VCA/13700 VCA.kicad_sch (KiCad schematic)
At the start: 65 parts, among them J101 Conn_02x05_Odd_Even, J102 AudioJack2_SwitchT, J103 AudioJack2_SwitchT, J104 AudioJack2_SwitchT, J105 AudioJack2_SwitchT, J106 AudioJack2_SwitchT, J107 AudioJack2_SwitchT, J108 AudioJack2_SwitchT, Q101 2N3906, Q102 2N3906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

Commit message: Create VCA front end project
Parts:
- J102, J103, J104, J105, J106, J107, J108: symbol Connector:AudioJack2_SwitchT -> Connector_Audio:AudioJack2_SwitchT
- Q101, Q102: footprint Package_TO_SOT_THT:TO-92_HandSolder -> Package_TO_SOT_THT:TO-92_Inline

Commit message: Finish VCA PCB
Parts:
- removed J102, J103, J104, J105, J106, J107, J108: AudioJack2_SwitchT, Connector_Audio:Jack_3.5mm_QingPu_WQP-PJ398SM_Vertical_CircularHoles, symbol Connector_Audio:AudioJack2_SwitchT
- removed R101, R102, R116, R117: 47k, Resistor_THT:R_Axial_DIN0207_L6.3mm_D2.5mm_P7.62mm_Horizontal, symbol Device:R
- removed R103, R118: 15k, Resistor_THT:R_Axial_DIN0207_L6.3mm_D2.5mm_P7.62mm_Horizontal, symbol Device:R
- removed R105, R108, R120, R123: 100k, Resistor_THT:R_Axial_DIN0207_L6.3mm_D2.5mm_P7.62mm_Horizontal, symbol Device:R
- removed RV101, RV102, RV104, RV105: 10k, 0_Potentiometer_THT:Potentiometer_Alpha_RD901F-40-00D_Single_Vertical_MP, symbol Device:R_Potentiometer_MountingPin
- added H1, H2: MNT_STANDOFF, 0_MountingHole:MountingHole_Pitch7.5mm_Drill3.4mm, symbol Mechanical:MountingHole_Pad
- added J2: Conn_01x19, Connector_PinHeader_2.54mm:PinHeader_1x19_P2.54mm_Vertical, symbol Connector_Generic:Conn_01x19
- J101: symbol Connector_Generic:Conn_02x05_Odd_Even -> Connector_Generic:Conn_02x05_Top_Bottom
- Q101, Q102: footprint Package_TO_SOT_THT:TO-92_Inline -> Package_TO_SOT_THT:TO-92_HandSolder
Connections:
- net +12V: now also J101.6 (Pin_6), J2.10 (Pin_10); no longer J101.2 (Pin_2)
- net -12V: now also J101.5 (Pin_5), J2.11 (Pin_11); no longer J101.9 (Pin_9)
- net Chassis: now also J101.3 (Pin_3), J101.8 (Pin_8), J2.12 (Pin_12), J2.13 (Pin_13), J2.14 (Pin_14), J2.15 (Pin_15); no longer J101.5 (Pin_5), J101.6 (Pin_6)
- net GND: now also J101.2 (Pin_2), J101.9 (Pin_9), J2.6 (Pin_6), J2.7 (Pin_7), J2.8 (Pin_8), J2.9 (Pin_9); no longer J101.3 (Pin_3), J101.8 (Pin_8)
- net OUT_2: now reaches R129.2, R130.2
- net OUT_2: now also J2.17 (Pin_17)
- net CV_2: now reaches C111.1, D104.1 (K), R121.2, R122.2, R124.2, R126.1, U102.6 (-)
- net CV_2: now also J2.5 (Pin_5)
- net CV_1: now reaches C103.1, D103.1 (K), R106.2, R107.2, R109.2, R111.1, U102.2 (-)
- net CV_1: now also J2.1 (Pin_1)
- net IN_2: now reaches RV106.1, U101.4 (-)
- net IN_2: now also J2.19 (Pin_19)
- net IN_1: now reaches RV103.1, U101.13 (-)
- net IN_1: now also J2.18 (Pin_18)
- net OUT_1: now reaches R114.2, R115.2
- net OUT_1: now also J2.16 (Pin_16)
- net Stereo Controls/CV_COMMON renamed CV_COMMON
- net CV_COMMON: now also J2.2 (Pin_2)
- net Stereo Controls/CV_COMMON_OFFSET renamed CV_COMMON_OFFSET
- net CV_COMMON_OFFSET: now also J2.3 (Pin_3)
- new net PAN_CV: J2.4 (Pin_4)
- no-connect marks 9 -> 4
Other:
- sheet Stereo Controls ports: added PAN_CV; removed CV_COMMON, CV_COMMON_OFFSET
- moved on the sheet: C101, C102, C103, C104, C105, C106, C107, C108, C109, C110, C111, C112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

Commit message: New VCLPF and Out
Parts:
- J101: value Conn_02x05_Odd_Even -> Conn_02x05_Top_Bottom
Changed lines of the file:
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@@
 			)
 		)
-		(property "Value" "Conn_02x05_Odd_Even"
+		(property "Value" "Conn_02x05_Top_Bottom"
 			(at 21.59 177.8 90)
 			(effects

Commit message: Begin revised delay
Parts:
- added C201, C204: 1n, 0_Capacitor_THT:C_Disc_D5.5mm_W2.5mm_P2.50mm, symbol Device:C
- added C202, C203: 0.1u, 0_Capacitor_THT:C_Disc_D5.5mm_W2.5mm_P2.50mm, symbol Device:C
- added R203: 56k, Resistor_THT:R_Axial_DIN0207_L6.3mm_D2.5mm_P7.62mm_Horizontal, symbol Device:R
- added R204, R205: 4.7k, Resistor_THT:R_Axial_DIN0207_L6.3mm_D2.5mm_P7.62mm_Horizontal, symbol Device:R
- added R4, R5: 47k, Resistor_THT:R_Axial_DIN0207_L6.3mm_D2.5mm_P7.62mm_Horizontal, symbol Device:R
- added U201: TL072, Package_DIP:DIP-8_W7.62mm_Socket, symbol Amplifier_Operational:TL072
Connections:
- net +12V: now also C202.2, U201.8 (V+)
- net -12V: now also C203.1, U201.4 (V-)
- net GND: now also C202.1, C203.2, U201.3 (+), U201.5 (+)
- net IN_1: now also R4.1; no longer RV103.1, U101.13 (-)
- net IN_2: now also R5.1; no longer RV106.1, U101.4 (-)
- net PAN_CV: now also C201.1, R203.1, U201.2 (-)
- net Stereo Controls/PAN_1: no longer names the net of R106.1
- net Stereo Controls/PAN_1: now also C201.2, R203.2, R204.1, U201.1
- net Stereo Controls/PAN_2: no longer names the net of R121.1
- net Stereo Controls/PAN_2: now also C204.2, R205.2, U201.7
- new net: C204.1, R204.2, R205.1, U201.6 (-)
- new net: R5.2, RV106.1, U101.4 (-)
- new net: R4.2, RV103.1, U101.13 (-)
Other:
- removed sheet Stereo Controls
- moved on the sheet: C103, C106, C107, C108, C109, C110, C111, C112, D103, D104, H1, H2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
