File: VCLPF/VCLPF.kicad_sch (KiCad schematic)
At the start: 60 parts, among them J1 Conn_01x15_Socket, J2 Conn_02x05_Top_Bottom, Q1 2N3904, Q10 2N3904, Q11 2N3904, Q12 2N3904, Q2 2N3904, Q3 2N3904, Q4 2N3904, Q5 2N3904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

Commit message: Begin revised delay
Parts:
- R5: value 100 -> 390
Changed lines of the file:
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@@
 			)
 		)
-		(property "Value" "100"
+		(property "Value" "390"
 			(at 93.218 119.253 0)
 			(effects
