File: Delay/Front End/Front End.kicad_sch (KiCad schematic)
At the start: 16 parts, among them J1 Conn_01x10_Pin, J2 AudioJack2_SwitchT, J3 AudioJack2_SwitchT, J4 AudioJack2_SwitchT, J5 AudioJack2_SwitchT, J6 AudioJack2_SwitchT

Commit message: Begin revised delay
Parts:
- removed J1: Conn_01x10_Pin, Connector_PinSocket_2.54mm:PinSocket_1x10_P2.54mm_Vertical, symbol Connector:Conn_01x10_Socket
- removed J4, J5, J6: AudioJack2_SwitchT, Connector_Audio:Jack_3.5mm_QingPu_WQP-PJ398SM_Vertical_CircularHoles, symbol Connector_Audio:AudioJack2_SwitchT
- removed R3, R4: 100k, Resistor_THT:R_Axial_DIN0207_L6.3mm_D2.5mm_P7.62mm_Horizontal, symbol Device:R
- removed RV4: 10k, 0_Potentiometer_THT:Potentiometer_Alpha_RD901F-40-00D_Single_Vertical_MP, symbol Device:R_Potentiometer_MountingPin
- added J1: AudioJack2_SwitchT, Connector_Audio:Jack_3.5mm_QingPu_WQP-PJ398SM_Vertical_CircularHoles, symbol Connector_Audio:AudioJack2_SwitchT
- added J4: Conn_01x14_Socket, Connector_PinHeader_2.54mm:PinHeader_1x14_P2.54mm_Vertical, symbol Connector:Conn_01x14_Socket
- R1, R2: value 100k -> 150k
- RV1: value 10k -> 50k
Connections:
- net Chassis: now also J1.S, J4.10 (Pin_10), J4.11 (Pin_11), J4.12 (Pin_12), J4.9 (Pin_9)
- net GND: now also J4.5 (Pin_5), J4.6 (Pin_6), J4.7 (Pin_7), J4.8 (Pin_8)
- net OUT: now also J3.T, J4.14 (Pin_14)
- net at RV2.3: now also J1.T; no longer J3.T
- net at RV3.2: now also R2.2
- net FB_3: now reaches RV1.3
- net FB_3: now also J4.3 (Pin_3); no longer J2.T
- net at RV2.2: now also R1.2; no longer R2.1
- net +12V: now reaches RV3.3
- net +12V: now also J4.1 (Pin_1)
- net FB_2: now reaches RV1.2
- net FB_2: now also J4.4 (Pin_4); no longer R1.1
- removed net MIX_IN: R1.2, R2.2
- new net IN: J2.T, J4.13 (Pin_13)
- new net TIME: J4.2 (Pin_2), R1.1, R2.1
- no-connect marks 7 -> 5

Commit message: PCB fixes and cleanup
Changed lines of the file:
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@@
 (kicad_sch
-	(version 20231120)
+	(version 20250114)
 	(generator "eeschema")
-	(generator_version "8.0")
+	(generator_version "9.0")
 	(paper "A4")
 	(junction
@@
 	(label "FB_2"
 		(at 63.5 83.82 0)
-		(fields_autoplaced yes)
 		(effects
 			(font
@@
 	(label "TIME"
 		(at 88.9 48.26 0)
-		(fields_autoplaced yes)
 		(effects
 			(font
@@
 	(label "IN"
 		(at 114.3 111.76 180)
-		(fields_autoplaced yes)
 		(effects
 			(font
@@
 	(label "TIME"
 		(at 114.3 83.82 180)
-		(fields_autoplaced yes)
 		(effects
 			(font
@@
 	(label "IN"
 		(at 64.77 109.22 0)
-		(fields_autoplaced yes)
 		(effects
 			(font
@@
 	(label "FB_3"
 		(at 114.3 86.36 180)
-		(fields_autoplaced yes)
 		(effects
 			(font
@@
 	(label "OUT"
 		(at 49.53 128.27 0)
-		(fields_autoplaced yes)
 		(effects
 			(font
@@
 	(label "FB_3"
 		(at 59.69 80.01 0)
-		(fields_autoplaced yes)
 		(effects
 			(font
@@
 	(label "OUT"
 		(at 114.3 114.3 180)
-		(fields_autoplaced yes)
 		(effects
 			(font
@@
 	(label "FB_2"
 		(at 114.3 88.9 180)
-		(fields_autoplaced yes)
 		(effects
 			(font
@@
 		)
 	)
+	(embedded_fonts no)
 )
