File: Diode VCLPF/Diode VCLPF.kicad_pcb (KiCad board)
At the start: 2 copper layers, 50.5 x 104.5 mm, 80 parts, among them J1 Conn_02x05_Top_Bottom, J2 Conn_01x15_Socket, Q1 2N3904, Q10 2N3904, Q11 2N3904, Q12 2N3904, Q13 2N3906, Q14 2N3904, Q2 2N3904, Q3 2N3904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

Commit message: PCB fixes and cleanup
Connections:
- C21 pad 2: Net-(U3-A) -> GND
- R28 pad 2: Net-(U3-A) -> GND
- U3 pad 2: Net-(U3-A) -> GND
Routing:
- net Net-(U3-A): track 13.0 -> 0.00 mm
- net Net-(U3-REF): vias 2 -> 0
