File: Diode VCLPF/Diode VCLPF.kicad_sch (KiCad schematic)
At the start: 80 parts, among them J1 Conn_02x05_Top_Bottom, J2 Conn_01x15_Socket, Q1 2N3904, Q10 2N3904, Q11 2N3904, Q12 2N3904, Q13 2N3906, Q14 2N3904, Q2 2N3904, Q3 2N3904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

Commit message: PCB fixes and cleanup
Connections:
- net GND: now also C21.2, R28.2, U3.2 (A)
Changed lines of the file:
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@@
 (kicad_sch
-	(version 20231120)
+	(version 20250114)
 	(generator "eeschema")
-	(generator_version "8.0")
+	(generator_version "9.0")
 	(paper "A4")
 	(junction
@@
 	(label "RES_2"
 		(at 260.35 87.63 180)
-		(fields_autoplaced yes)
 		(effects
 			(font
@@
 	(label "IN"
 		(at 260.35 95.25 180)
-		(fields_autoplaced yes)
 		(effects
 			(font
@@
 	(label "OUT"
 		(at 260.35 97.79 180)
-		(fields_autoplaced yes)
 		(effects
 			(font
@@
 	(label "OUT"
 		(at 203.2 74.93 0)
-		(fields_autoplaced yes)
 		(effects
 			(font
@@
 	(label "5.333V"
 		(at 274.32 31.75 0)
-		(fields_autoplaced yes)
 		(effects
 			(font
@@
 	(label "RES_3"
 		(at 260.35 90.17 180)
-		(fields_autoplaced yes)
 		(effects
 			(font
@@
 	(label "IN"
 		(at 38.1 90.17 0)
-		(fields_autoplaced yes)
 		(effects
 			(font
@@
 	(label "CV"
 		(at 148.59 171.45 0)
-		(fields_autoplaced yes)
 		(effects
 			(font
@@
 	(label "GAIN_1"
 		(at 203.2 78.74 180)
-		(fields_autoplaced yes)
 		(effects
 			(font
@@
 	(label "5.333V"
 		(at 49.53 157.48 90)
-		(fields_autoplaced yes)
 		(effects
 			(font
@@
 	(label "RES_2"
 		(at 165.1 97.79 0)
-		(fields_autoplaced yes)
 		(effects
 			(font
@@
 	(label "5.333V"
 		(at 139.7 107.95 90)
-		(fields_autoplaced yes)
 		(effects
 			(font
@@
 	(label "GAIN_1"
 		(at 260.35 92.71 180)
-		(fields_autoplaced yes)
 		(effects
 			(font
@@
 	(label "5.333V"
 		(at 38.1 120.65 90)
-		(fields_autoplaced yes)
 		(effects
 			(font
@@
 	(label "RES_3"
 		(at 165.1 93.98 0)
-		(fields_autoplaced yes)
 		(effects
 			(font
@@
 	(label "CV"
 		(at 260.35 82.55 180)
-		(fields_autoplaced yes)
 		(effects
 			(font
@@
 	)
 	(symbol
+		(lib_id "power:GND")
+		(at 257.81 60.96 0)
+		(unit 1)
+		(exclude_from_sim no)
+		(in_bom yes)
+		(on_board yes)
+		(dnp no)
+		(fields_autoplaced yes)
+		(property "Reference" "#PWR032"
+			(at 257.81 67.31 0)
+			(effects
+				(font
+					(size 1.27 1.27)
+				)
+				(hide yes)
+			)
+		)
+		(property "Value" "GND"
+			(at 257.81 66.04 0)
+			(effects
+				(font
+					(size 1.27 1.27)
+				)
+			)
+		)
+		(property "Footprint" ""
+			(at 257.81 60.96 0)
+			(effects
+				(font
+					(size 1.27 1.27)
+				)
+				(hide yes)
+			)
+		)
+		(property "Datasheet" ""
+			(at 257.81 60.96 0)
+			(effects
+				(font
+					(size 1.27 1.27)
+				)
+				(hide yes)
+			)
+		)
+		(property "Description" "Power symbol creates a global label with name \"GND\" , ground"
+			(at 257.81 60.96 0)
+			(effects
+				(font
+					(size 1.27 1.27)
+				)
+				(hide yes)
+			)
+		)
+		(pin "1"
+		)
+		(instances
+			(project "Diode VCLPF"
+				(path "/acdb742a-b610-48fa-ba53-3f9a9d7426f3"
+					(reference "#PWR032")
+					(unit 1)
+				)
+			)
+		)
+	)
+	(symbol
 		(lib_id "Device:R")
 		(at 138.43 166.37 270)
@@
 		)
 	)
+	(embedded_fonts no)
 )
