File: Envelope Generator/Front End/Front End.kicad_pcb (KiCad board)
At the start: 2 copper layers, 50.5 x 104.5 mm, 13 parts, among them J101 AudioJack2_SwitchT, J102 AudioJack2_SwitchT, J103 AudioJack2_SwitchT, J104 Conn_01x23, SW101 SW_SPST, SW102 SW_SPDT

Commit message: New VCLPF and Out
Parts:
- J104: moved to B.Cu
- turned J104 to 180 degrees
Other:
- board text added: "JLCJLCJLCJLC"
