File: Minimal SVVCF/Front End/Front End.kicad_pcb (KiCad board)
At the start: 2 copper layers, 40.3 x 104.5 mm, 16 parts, among them J1 AudioJack2_SwitchT, J2 AudioJack2_SwitchT, J3 AudioJack2_SwitchT, J4 AudioJack2_SwitchT, J5 AudioJack2_SwitchT, J6 AudioJack2_SwitchT, J7 Conn_01x16_Socket

Commit message: PCB fixes and cleanup
Connections:
- J7 pad 2: GND -> -12V
- RV3 pad 1: GND -> -12V
Routing:
- net -12V: track 0.00 -> 38.2 mm, vias 0 -> 2
- net GND: track 83.6 -> 55.8 mm
