File: Mixer/Front End/Front End.kicad_pcb (KiCad board)
At the start: 2 copper layers, 40.3 x 104.5 mm, 16 parts, among them J1 Conn_01x10_Pin, J2 AudioJack2_SwitchT, J3 AudioJack2_SwitchT, J4 AudioJack2_SwitchT, J5 AudioJack2_SwitchT, J6 AudioJack2_SwitchT

Commit message: Begin revised delay
Connections:
- J6 pad T: (no net) -> /OUT
Changed lines of the file:
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@@
 			)
 		)
+		(property ki_fp_filters "Jack*")
+		(sheetname "Root")
+		(sheetfile "Front End.kicad_sch")
 		(attr through_hole)
 		(fp_line
@@
 			(layers "*.Cu" "*.Mask")
 			(remove_unused_layers no)
+			(net 6 "/OUT")
 			(pintype "passive")
 		)
@@
 			)
 		)
+		(property ki_fp_filters "Potentiometer*")
+		(sheetname "Root")
+		(sheetfile "Front End.kicad_sch")
 		(attr through_hole)
 		(fp_line
@@
 			)
 		)
+		(property ki_fp_filters "Jack*")
+		(sheetname "Root")
+		(sheetfile "Front End.kicad_sch")
 		(attr through_hole)
 		(fp_line
@@
 			)
 		)
+		(property ki_fp_filters "Jack*")
+		(sheetname "Root")
+		(sheetfile "Front End.kicad_sch")
 		(attr through_hole)
 		(fp_line
@@
 			)
 		)
+		(property ki_fp_filters "Jack*")
+		(sheetname "Root")
+		(sheetfile "Front End.kicad_sch")
 		(attr through_hole)
 		(fp_line
@@
 			)
 		)
+		(property ki_fp_filters "Potentiometer*")
+		(sheetname "Root")
+		(sheetfile "Front End.kicad_sch")
 		(attr through_hole)
 		(fp_line
@@
 			)
 		)
+		(property ki_fp_filters "Potentiometer*")
+		(sheetname "Root")
+		(sheetfile "Front End.kicad_sch")
 		(attr through_hole)
 		(fp_line
@@
 			)
 		)
+		(property ki_fp_filters "Jack*")
+		(sheetname "Root")
+		(sheetfile "Front End.kicad_sch")
 		(attr through_hole)
 		(fp_line
@@
 			)
 		)
+		(property ki_fp_filters "Potentiometer*")
+		(sheetname "Root")
+		(sheetfile "Front End.kicad_sch")
 		(attr through_hole)
 		(fp_line

Commit message: PCB fixes and cleanup
Routing:
- net /OUT: track 0.00 -> 59.0 mm, vias 0 -> 1
