File: Mixer/Front End/Front End.kicad_sch (KiCad schematic)
At the start: 16 parts, among them J1 Conn_01x10_Pin, J2 AudioJack2_SwitchT, J3 AudioJack2_SwitchT, J4 AudioJack2_SwitchT, J5 AudioJack2_SwitchT, J6 AudioJack2_SwitchT

Commit message: PCB fixes and cleanup
Changed lines of the file:
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@@
 (kicad_sch
-	(version 20231120)
+	(version 20250114)
 	(generator "eeschema")
-	(generator_version "8.0")
+	(generator_version "9.0")
 	(paper "A4")
 	(junction
@@
 	(label "MIX_IN"
 		(at 179.07 92.71 0)
-		(fields_autoplaced yes)
 		(effects
 			(font
@@
 	(label "OUT"
 		(at 200.66 92.71 180)
-		(fields_autoplaced yes)
 		(effects
 			(font
@@
 	(label "MIX_IN"
 		(at 104.14 80.01 180)
-		(fields_autoplaced yes)
 		(effects
 			(font
@@
 	(label "OUT"
 		(at 102.87 82.55 180)
-		(fields_autoplaced yes)
 		(effects
 			(font
@@
 		)
 	)
+	(embedded_fonts no)
 )
